File: 1 - Main System/KiCAD Project Files/Headless.kicad_sch (KiCad schematic)
At the start: 0 parts

Commit message: Routing DDR3 Completed (pre-review)
Other:
- sheet FPGA Power Distro ports: added +0V674, +0V674_REF; removed none
Changed lines of the file:
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@@
 	(sheet
 		(at 107.95 129.54)
-		(size 39.37 24.13)
+		(size 39.37 25.4)
 		(exclude_from_sim no)
 		(in_bom yes)
@@
 		)
 		(property "Sheetfile" "fpga_zynq.kicad_sch"
-			(at 107.95 154.2546 0)
+			(at 107.95 155.5246 0)
 			(show_name no)
 			(do_not_autoplace no)
@@
 	(sheet
 		(at 68.58 129.54)
-		(size 19.05 17.78)
+		(size 19.05 25.4)
 		(exclude_from_sim no)
 		(in_bom yes)
@@
 		)
 		(property "Sheetfile" "fpgapowdistro.kicad_sch"
-			(at 68.58 147.9046 0)
+			(at 68.58 155.5246 0)
 			(show_name no)
 			(do_not_autoplace no)
@@
 			(effects
 				(font
+					(size 1.27 1.27)
+				)
+				(justify right)
+			)
+		)
+		(pin "+0V674_REF" output
+			(at 87.63 149.86 0)
+			(effects
+				(font
+					(size 1.27 1.27)
+				)
+				(justify right)
+			)
+		)
+		(pin "+0V674" output
+			(at 87.63 152.4 0)
+			(effects
+				(font
